Commit message: model of hospital

File: src/pickplace_arm_description/urdf/pickplace_arm.gazebo.xacro (robot description, xacro)
@@ -149,21 +149,35 @@
        NOT a nicety: without it the robot tows all three boxes off the table
        the moment it drives to the pick. -->
-  <xacro:macro name="box_attach" params="color">
+  <xacro:macro name="grasp_attach" params="model">
     <gazebo>
       <plugin filename="gz-sim-detachable-joint-system"
               name="gz::sim::systems::DetachableJoint">
         <parent_link>fr3_link7</parent_link>
-        <child_model>box_${color}</child_model>
+        <child_model>${model}</child_model>
         <child_link>link</child_link>
-        <attach_topic>/box_${color}/attach</attach_topic>
-        <detach_topic>/box_${color}/detach</detach_topic>
-        <output_topic>/box_${color}/attach_state</output_topic>
+        <attach_topic>/${model}/attach</attach_topic>
+        <detach_topic>/${model}/detach</detach_topic>
+        <output_topic>/${model}/attach_state</output_topic>
         <suppress_child_warning>true</suppress_child_warning>
       </plugin>
     </gazebo>
   </xacro:macro>
-  <xacro:box_attach color="red"/>
-  <xacro:box_attach color="green"/>
-  <xacro:box_attach color="blue"/>
+  <xacro:grasp_attach model="box_red"/>
+  <xacro:grasp_attach model="box_green"/>
+  <xacro:grasp_attach model="box_blue"/>
+  <!-- Blood sample rack, the payload of the hospital lab -> ward run. Same
+       rigid-grasp treatment as the boxes, for a stronger reason: this payload
+       is carried the length of a corridor rather than a few metres across a
+       room, so any friction-held grip has that much longer to creep. The rack's
+       grip block is a 0.06 m cube, the same size the boxes present to the
+       jaws, so the grasp itself is verified by the existing finger-gap check.
+       This model is only ever spawned for the hospital mission. The plugin
+       tolerates its absence - suppress_child_warning keeps the log clean when
+       the warehouse mission runs and no sample_rack exists.
+       The startup-detach caveat above applies here too: the joint is created
+       the instant the rack spawns, so the mission MUST publish
+       /sample_rack/detach before driving off, or the robot drags the rack off
+       the bench with it. -->
+  <xacro:grasp_attach model="sample_rack"/>
   <!-- High friction + soft contact on the finger pads so the gripper can
        actually hold a box by friction in Gazebo Harmonic. Raised 3.5 -> 5.0

Commit message: the first plane

File: src/pickplace_arm_description/urdf/pickplace_arm.gazebo.xacro (robot description, xacro)
@@ -121,5 +121,11 @@
       <parameters>$(find pickplace_arm_description)/config/arm_controllers.yaml</parameters>
       <ros>
-        <remapping>~/robot_description:=/robot_description</remapping>
+        <!-- Emitted only when robot_ns is set. An empty <namespace/> is not the
+             same as no namespace to the plugin, so the single-robot SDF has to
+             come out with this element absent, exactly as before. -->
+        <xacro:if value="${robot_ns != ''}">
+          <namespace>${robot_ns}</namespace>
+        </xacro:if>
+        <remapping>~/robot_description:=${ns_topic}/robot_description</remapping>
       </ros>
     </plugin>
@@ -156,7 +162,7 @@
         <child_model>${model}</child_model>
         <child_link>link</child_link>
-        <attach_topic>/${model}/attach</attach_topic>
-        <detach_topic>/${model}/detach</detach_topic>
-        <output_topic>/${model}/attach_state</output_topic>
+        <attach_topic>${ns_topic}/${model}/attach</attach_topic>
+        <detach_topic>${ns_topic}/${model}/detach</detach_topic>
+        <output_topic>${ns_topic}/${model}/attach_state</output_topic>
         <suppress_child_warning>true</suppress_child_warning>
       </plugin>
@@ -225,5 +231,5 @@
   <gazebo reference="camera_link">
     <sensor name="rgbd_camera" type="rgbd_camera">
-      <topic>/camera</topic>
+      <topic>${ns_topic}/camera</topic>
       <!-- 5 Hz, down from 30. RGB-D rendering is BY FAR the most expensive
            thing in this simulation: two 640x480 rgbd_camera sensors at 30 Hz
@@ -272,5 +278,5 @@
            i.e. unambiguously X-forward. See the front camera below for the
            same fix and the reason nothing else changes. -->
-      <gz_frame_id>camera_link</gz_frame_id>
+      <gz_frame_id>${ns_frame}camera_link</gz_frame_id>
     </sensor>
   </gazebo>
@@ -278,5 +284,5 @@
   <gazebo reference="lidar_link">
     <sensor name="lidar" type="gpu_lidar">
-      <topic>/scan</topic>
+      <topic>${ns_topic}/scan</topic>
       <update_rate>10</update_rate>
       <always_on>1</always_on>
@@ -308,5 +314,5 @@
         </noise>
       </lidar>
-      <gz_frame_id>lidar_link</gz_frame_id>
+      <gz_frame_id>${ns_frame}lidar_link</gz_frame_id>
     </sensor>
   </gazebo>
@@ -315,8 +321,8 @@
   <gazebo reference="imu_link">
     <sensor name="imu" type="imu">
-      <topic>/imu</topic>
+      <topic>${ns_topic}/imu</topic>
       <update_rate>50</update_rate>
       <always_on>1</always_on>
-      <gz_frame_id>imu_link</gz_frame_id>
+      <gz_frame_id>${ns_frame}imu_link</gz_frame_id>
     </sensor>
   </gazebo>
@@ -324,5 +330,5 @@
   <gazebo reference="front_camera_link">
     <sensor name="front_rgbd_camera" type="rgbd_camera">
-      <topic>/front_camera</topic>
+      <topic>${ns_topic}/front_camera</topic>
       <!-- 15 Hz, down from 30 - see the wrist camera above for the measured
            cost. This one carries the whole mission (box pick AND column
@@ -372,5 +378,5 @@
            need one (depth_image_proc and friends assume that convention), and
            removing it would break nothing but document nothing either. -->
-      <gz_frame_id>front_camera_link</gz_frame_id>
+      <gz_frame_id>${ns_frame}front_camera_link</gz_frame_id>
     </sensor>
   </gazebo>

File: src/pickplace_arm_description/urdf/pickplace_arm.urdf.xacro (robot description, xacro)
@@ -52,4 +52,24 @@
   <xacro:arg name="is_sim" default="false"/>
   <xacro:arg name="use_platform_controllers" default="false"/>
+  <!-- MULTI-ROBOT. Empty by default, and every use of it below is written so
+       that empty reproduces the single-robot description EXACTLY - the
+       missions that spawn one robot are unaffected by this arg existing.
+       Set it (e.g. robot_ns:=r1) and the description becomes one of several
+       that can share a world:
+         sensor topics    /scan           -> /r1/scan
+         sensor frames    lidar_link      -> r1/lidar_link
+         grasp topics     /box_red/attach -> /r1/box_red/attach
+         controller node  /controller_manager -> /r1/controller_manager
+       LINK NAMES ARE DELIBERATELY NOT PREFIXED. They are referenced by the
+       MoveIt config, the ros2_control joint list, the DetachableJoint's
+       parent_link and the Clearpath/Franka includes; prefixing them would mean
+       touching all of those. Gazebo scopes links by model name already, and the
+       TF tree is separated by robot_state_publisher's frame_prefix - which is
+       exactly what the prefixed sensor frames above are matched to. -->
+  <xacro:arg name="robot_ns" default=""/>
+  <xacro:property name="robot_ns" value="$(arg robot_ns)"/>
+  <!-- '' or '/r1' for topic names; '' or 'r1/' for frame ids. -->
+  <xacro:property name="ns_topic" value="${'' if robot_ns == '' else '/' + robot_ns}"/>
+  <xacro:property name="ns_frame" value="${'' if robot_ns == '' else robot_ns + '/'}"/>
   <xacro:property name="PI" value="3.14159265359"/>
   <!-- Materials for the sensor housings we add ourselves (the A200 and FR3

Commit message: Brought all the changes back from main

File: src/pickplace_arm_description/urdf/pickplace_arm.gazebo.xacro (robot description, xacro)
@@ -121,11 +121,5 @@
       <parameters>$(find pickplace_arm_description)/config/arm_controllers.yaml</parameters>
       <ros>
-        <!-- Emitted only when robot_ns is set. An empty <namespace/> is not the
-             same as no namespace to the plugin, so the single-robot SDF has to
-             come out with this element absent, exactly as before. -->
-        <xacro:if value="${robot_ns != ''}">
-          <namespace>${robot_ns}</namespace>
-        </xacro:if>
-        <remapping>~/robot_description:=${ns_topic}/robot_description</remapping>
+        <remapping>~/robot_description:=/robot_description</remapping>
       </ros>
     </plugin>
@@ -155,35 +149,21 @@
        NOT a nicety: without it the robot tows all three boxes off the table
        the moment it drives to the pick. -->
-  <xacro:macro name="grasp_attach" params="model">
+  <xacro:macro name="box_attach" params="color">
     <gazebo>
       <plugin filename="gz-sim-detachable-joint-system"
               name="gz::sim::systems::DetachableJoint">
         <parent_link>fr3_link7</parent_link>
-        <child_model>${model}</child_model>
+        <child_model>box_${color}</child_model>
         <child_link>link</child_link>
-        <attach_topic>${ns_topic}/${model}/attach</attach_topic>
-        <detach_topic>${ns_topic}/${model}/detach</detach_topic>
-        <output_topic>${ns_topic}/${model}/attach_state</output_topic>
+        <attach_topic>/box_${color}/attach</attach_topic>
+        <detach_topic>/box_${color}/detach</detach_topic>
+        <output_topic>/box_${color}/attach_state</output_topic>
         <suppress_child_warning>true</suppress_child_warning>
       </plugin>
     </gazebo>
   </xacro:macro>
-  <xacro:grasp_attach model="box_red"/>
-  <xacro:grasp_attach model="box_green"/>
-  <xacro:grasp_attach model="box_blue"/>
-  <!-- Blood sample rack, the payload of the hospital lab -> ward run. Same
-       rigid-grasp treatment as the boxes, for a stronger reason: this payload
-       is carried the length of a corridor rather than a few metres across a
-       room, so any friction-held grip has that much longer to creep. The rack's
-       grip block is a 0.06 m cube, the same size the boxes present to the
-       jaws, so the grasp itself is verified by the existing finger-gap check.
-       This model is only ever spawned for the hospital mission. The plugin
-       tolerates its absence - suppress_child_warning keeps the log clean when
-       the warehouse mission runs and no sample_rack exists.
-       The startup-detach caveat above applies here too: the joint is created
-       the instant the rack spawns, so the mission MUST publish
-       /sample_rack/detach before driving off, or the robot drags the rack off
-       the bench with it. -->
-  <xacro:grasp_attach model="sample_rack"/>
+  <xacro:box_attach color="red"/>
+  <xacro:box_attach color="green"/>
+  <xacro:box_attach color="blue"/>
   <!-- High friction + soft contact on the finger pads so the gripper can
        actually hold a box by friction in Gazebo Harmonic. Raised 3.5 -> 5.0
@@ -215,7 +195,6 @@
   <xacro:macro name="wheel_friction" params="link">
     <gazebo reference="${link}">
-      <mu1>4.0</mu1>
-      <mu2>0.2</mu2>
-      <fdir1>1 0 0</fdir1>
+      <mu1>1.0</mu1>
+      <mu2>1.0</mu2>
       <kp>1e6</kp>
       <kd>1.0</kd>
@@ -232,5 +211,5 @@
   <gazebo reference="camera_link">
     <sensor name="rgbd_camera" type="rgbd_camera">
-      <topic>${ns_topic}/camera</topic>
+      <topic>/camera</topic>
       <!-- 5 Hz, down from 30. RGB-D rendering is BY FAR the most expensive
            thing in this simulation: two 640x480 rgbd_camera sensors at 30 Hz
@@ -279,5 +258,5 @@
            i.e. unambiguously X-forward. See the front camera below for the
            same fix and the reason nothing else changes. -->
-      <gz_frame_id>${ns_frame}camera_link</gz_frame_id>
+      <gz_frame_id>camera_link</gz_frame_id>
     </sensor>
   </gazebo>
@@ -285,5 +264,5 @@
   <gazebo reference="lidar_link">
     <sensor name="lidar" type="gpu_lidar">
-      <topic>${ns_topic}/scan</topic>
+      <topic>/scan</topic>
       <update_rate>10</update_rate>
       <always_on>1</always_on>
@@ -306,30 +285,5 @@
         <range>
           <min>0.12</min>
-          <!-- 25 m, NOT 8. THE OLD 8 WAS SHORTER THAN THE BUILDING.
-               The AWS hospital's north-south corridor is a 40.8 m straight run
-               of parallel wall (measured off this package's own map, y -25.95
-               to 14.85 along x = 4.5). A sensor that reaches 8 m into it sees
-               two walls and nothing else, and sees exactly the same two walls
-               from anywhere in the middle 25 m of it - so the scan carries no
-               information at all about position ALONG the corridor, which is
-               the one axis that matters there.
-               That is what was breaking localisation, and it was breaking it in
-               a way no amount of filter tuning could reach: alpha1-4,
-               recovery_alpha_* and the z_hit/z_rand pairing were each tried and
-               each failed, because all three are downstream of information the
-               sensor never delivered. Measured on the failing run, with
-               odometry perfectly healthy (d_odom 4.299 against d_truth 4.296 -
-               the wheels were NOT slipping): the robot travelled 4.3 m down
-               that corridor while AMCL's belief advanced 0.33 m, ending 4.6 m
-               behind the truth.
-               25 m puts both ends of that corridor in view from most of its
-               length, which is precisely the measurement that pins position
-               along the axis. It is also a real device spec rather than an
-               invented one - a SICK TiM781 reaches 25 m where the TiM551 this
-               was modelled on reaches 10 - so the sensor stays plausible.
-               amcl_tugbot.yaml's laser_max_range MUST be raised to match: AMCL
-               discards returns beyond its own limit, so leaving it at 8 would
-               throw away exactly the beams this change exists to provide. -->
-          <max>25.0</max>
+          <max>8.0</max>
           <resolution>0.01</resolution>
         </range>
@@ -340,5 +294,5 @@
         </noise>
       </lidar>
-      <gz_frame_id>${ns_frame}lidar_link</gz_frame_id>
+      <gz_frame_id>lidar_link</gz_frame_id>
     </sensor>
   </gazebo>
@@ -347,8 +301,8 @@
   <gazebo reference="imu_link">
     <sensor name="imu" type="imu">
-      <topic>${ns_topic}/imu</topic>
+      <topic>/imu</topic>
       <update_rate>50</update_rate>
       <always_on>1</always_on>
-      <gz_frame_id>${ns_frame}imu_link</gz_frame_id>
+      <gz_frame_id>imu_link</gz_frame_id>
     </sensor>
   </gazebo>
@@ -356,5 +310,5 @@
   <gazebo reference="front_camera_link">
     <sensor name="front_rgbd_camera" type="rgbd_camera">
-      <topic>${ns_topic}/front_camera</topic>
+      <topic>/front_camera</topic>
       <!-- 15 Hz, down from 30 - see the wrist camera above for the measured
            cost. This one carries the whole mission (box pick AND column
@@ -404,5 +358,5 @@
            need one (depth_image_proc and friends assume that convention), and
            removing it would break nothing but document nothing either. -->
-      <gz_frame_id>${ns_frame}front_camera_link</gz_frame_id>
+      <gz_frame_id>front_camera_link</gz_frame_id>
     </sensor>
   </gazebo>

File: src/pickplace_arm_description/urdf/pickplace_arm.urdf.xacro (robot description, xacro)
@@ -52,24 +52,4 @@
   <xacro:arg name="is_sim" default="false"/>
   <xacro:arg name="use_platform_controllers" default="false"/>
-  <!-- MULTI-ROBOT. Empty by default, and every use of it below is written so
-       that empty reproduces the single-robot description EXACTLY - the
-       missions that spawn one robot are unaffected by this arg existing.
-       Set it (e.g. robot_ns:=r1) and the description becomes one of several
-       that can share a world:
-         sensor topics    /scan           -> /r1/scan
-         sensor frames    lidar_link      -> r1/lidar_link
-         grasp topics     /box_red/attach -> /r1/box_red/attach
-         controller node  /controller_manager -> /r1/controller_manager
-       LINK NAMES ARE DELIBERATELY NOT PREFIXED. They are referenced by the
-       MoveIt config, the ros2_control joint list, the DetachableJoint's
-       parent_link and the Clearpath/Franka includes; prefixing them would mean
-       touching all of those. Gazebo scopes links by model name already, and the
-       TF tree is separated by robot_state_publisher's frame_prefix - which is
-       exactly what the prefixed sensor frames above are matched to. -->
-  <xacro:arg name="robot_ns" default=""/>
-  <xacro:property name="robot_ns" value="$(arg robot_ns)"/>
-  <!-- '' or '/r1' for topic names; '' or 'r1/' for frame ids. -->
-  <xacro:property name="ns_topic" value="${'' if robot_ns == '' else '/' + robot_ns}"/>
-  <xacro:property name="ns_frame" value="${'' if robot_ns == '' else robot_ns + '/'}"/>
   <xacro:property name="PI" value="3.14159265359"/>
   <!-- Materials for the sensor housings we add ourselves (the A200 and FR3

Commit message: Brought the new map (hospital), single robot, & no dyn. obstacle (yet), with the same main scenario

File: src/pickplace_arm_description/urdf/pickplace_arm.gazebo.xacro (robot description, xacro)
@@ -149,21 +149,29 @@
        NOT a nicety: without it the robot tows all three boxes off the table
        the moment it drives to the pick. -->
-  <xacro:macro name="box_attach" params="color">
+  <xacro:macro name="grasp_attach" params="model">
     <gazebo>
       <plugin filename="gz-sim-detachable-joint-system"
               name="gz::sim::systems::DetachableJoint">
         <parent_link>fr3_link7</parent_link>
-        <child_model>box_${color}</child_model>
+        <child_model>${model}</child_model>
         <child_link>link</child_link>
-        <attach_topic>/box_${color}/attach</attach_topic>
-        <detach_topic>/box_${color}/detach</detach_topic>
-        <output_topic>/box_${color}/attach_state</output_topic>
+        <attach_topic>/${model}/attach</attach_topic>
+        <detach_topic>/${model}/detach</detach_topic>
+        <output_topic>/${model}/attach_state</output_topic>
         <suppress_child_warning>true</suppress_child_warning>
       </plugin>
     </gazebo>
   </xacro:macro>
-  <xacro:box_attach color="red"/>
-  <xacro:box_attach color="green"/>
-  <xacro:box_attach color="blue"/>
+  <!-- The coloured boxes of the warehouse run. -->
+  <xacro:grasp_attach model="box_red"/>
+  <xacro:grasp_attach model="box_green"/>
+  <xacro:grasp_attach model="box_blue"/>
+  <!-- The sample racks of the hospital run. Declared unconditionally, exactly
+       like the boxes: suppress_child_warning is what makes a plugin whose child
+       model does not exist in this world harmless, so one robot description
+       serves both missions rather than needing a world-dependent URDF. -->
+  <xacro:grasp_attach model="rack_red"/>
+  <xacro:grasp_attach model="rack_green"/>
+  <xacro:grasp_attach model="rack_blue"/>
   <!-- High friction + soft contact on the finger pads so the gripper can
        actually hold a box by friction in Gazebo Harmonic. Raised 3.5 -> 5.0
