Commit message: Step 1: adding the 3 robots to the world and bringing them up

File: src/pickplace_arm_description/urdf/pickplace_arm.gazebo.xacro (robot description, xacro)
@@ -121,5 +121,11 @@
       <parameters>$(find pickplace_arm_description)/config/arm_controllers.yaml</parameters>
       <ros>
-        <remapping>~/robot_description:=/robot_description</remapping>
+        <!-- Emitted only when robot_ns is set. An empty <namespace/> is NOT the
+             same as no namespace to the plugin, so the single-robot SDF has to
+             come out with this element absent, exactly as before. -->
+        <xacro:if value="${robot_ns != ''}">
+          <namespace>${robot_ns}</namespace>
+        </xacro:if>
+        <remapping>~/robot_description:=${ns_topic}/robot_description</remapping>
       </ros>
     </plugin>
@@ -156,7 +162,7 @@
         <child_model>${model}</child_model>
         <child_link>link</child_link>
-        <attach_topic>/${model}/attach</attach_topic>
-        <detach_topic>/${model}/detach</detach_topic>
-        <output_topic>/${model}/attach_state</output_topic>
+        <attach_topic>${ns_topic}/${model}/attach</attach_topic>
+        <detach_topic>${ns_topic}/${model}/detach</detach_topic>
+        <output_topic>${ns_topic}/${model}/attach_state</output_topic>
         <suppress_child_warning>true</suppress_child_warning>
       </plugin>
@@ -219,5 +225,5 @@
   <gazebo reference="camera_link">
     <sensor name="rgbd_camera" type="rgbd_camera">
-      <topic>/camera</topic>
+      <topic>${ns_topic}/camera</topic>
       <!-- 5 Hz, down from 30. RGB-D rendering is BY FAR the most expensive
            thing in this simulation: two 640x480 rgbd_camera sensors at 30 Hz
@@ -266,5 +272,5 @@
            i.e. unambiguously X-forward. See the front camera below for the
            same fix and the reason nothing else changes. -->
-      <gz_frame_id>camera_link</gz_frame_id>
+      <gz_frame_id>${ns_frame}camera_link</gz_frame_id>
     </sensor>
   </gazebo>
@@ -272,5 +278,5 @@
   <gazebo reference="lidar_link">
     <sensor name="lidar" type="gpu_lidar">
-      <topic>/scan</topic>
+      <topic>${ns_topic}/scan</topic>
       <update_rate>10</update_rate>
       <always_on>1</always_on>
@@ -293,5 +299,32 @@
         <range>
           <min>0.12</min>
-          <max>8.0</max>
+          <!-- 25 m, NOT 8. THE OLD 8 WAS SHORTER THAN THE BUILDING.
+               Fine in the warehouse, which is small. In the AWS hospital the
+               north-south corridor is a 40.8 m straight run of parallel wall
+               (measured off this package's own map, y -25.95 to 14.85 along
+               x = 4.5). A sensor that reaches 8 m into it sees two walls and
+               nothing else, and sees exactly the SAME two walls from anywhere
+               in the middle 25 m of it - so the scan carries no information at
+               all about position ALONG the corridor, which is the one axis that
+               matters there.
+               That breaks localisation in a way no amount of filter tuning can
+               reach: alpha1-4, recovery_alpha_* and the z_hit/z_rand pairing
+               were each tried and each failed, because all three are downstream
+               of information the sensor never delivered. Measured on a failing
+               run, with odometry perfectly healthy (d_odom 4.299 against
+               d_truth 4.296 - the wheels were NOT slipping): the robot
+               travelled 4.3 m down that corridor while AMCL's belief advanced
+               0.33 m, ending 4.6 m behind the truth.
+               25 m puts both ends of that corridor in view from most of its
+               length, which is precisely the measurement that pins position
+               along the axis. It is also a real device spec rather than an
+               invented one - a SICK TiM781 reaches 25 m where the TiM551 this
+               was modelled on reaches 10 - so the sensor stays plausible.
+               AMCL's OWN laser_max_range MUST BE RAISED TO MATCH, or it
+               discards exactly the beams this exists to provide. Done in
+               amcl_hospital.yaml; amcl_tugbot.yaml deliberately stays at 8,
+               because the warehouse never had this problem and its numbers are
+               the ones that were tuned there. -->
+          <max>25.0</max>
           <resolution>0.01</resolution>
         </range>
@@ -302,5 +335,5 @@
         </noise>
       </lidar>
-      <gz_frame_id>lidar_link</gz_frame_id>
+      <gz_frame_id>${ns_frame}lidar_link</gz_frame_id>
     </sensor>
   </gazebo>
@@ -309,8 +342,8 @@
   <gazebo reference="imu_link">
     <sensor name="imu" type="imu">
-      <topic>/imu</topic>
+      <topic>${ns_topic}/imu</topic>
       <update_rate>50</update_rate>
       <always_on>1</always_on>
-      <gz_frame_id>imu_link</gz_frame_id>
+      <gz_frame_id>${ns_frame}imu_link</gz_frame_id>
     </sensor>
   </gazebo>
@@ -318,5 +351,5 @@
   <gazebo reference="front_camera_link">
     <sensor name="front_rgbd_camera" type="rgbd_camera">
-      <topic>/front_camera</topic>
+      <topic>${ns_topic}/front_camera</topic>
       <!-- 15 Hz, down from 30 - see the wrist camera above for the measured
            cost. This one carries the whole mission (box pick AND column
@@ -366,5 +399,5 @@
            need one (depth_image_proc and friends assume that convention), and
            removing it would break nothing but document nothing either. -->
-      <gz_frame_id>front_camera_link</gz_frame_id>
+      <gz_frame_id>${ns_frame}front_camera_link</gz_frame_id>
     </sensor>
   </gazebo>

File: src/pickplace_arm_description/urdf/pickplace_arm.urdf.xacro (robot description, xacro)
@@ -52,4 +52,25 @@
   <xacro:arg name="is_sim" default="false"/>
   <xacro:arg name="use_platform_controllers" default="false"/>
+  <!-- MULTI-ROBOT. Empty by default, and every use of it below is written so
+       that empty reproduces the single-robot description EXACTLY - the missions
+       that spawn one robot are unaffected by this arg existing. Set it (e.g.
+       robot_ns:=r1) and the description becomes one of several that can share a
+       world:
+         sensor topics    /scan            -> /r1/scan
+         sensor frames    lidar_link       -> r1/lidar_link
+         grasp topics     /rack_red/attach -> /r1/rack_red/attach
+         controller node  /controller_manager -> /r1/controller_manager
+       LINK NAMES ARE DELIBERATELY NOT PREFIXED. They are referenced by the
+       MoveIt config, the ros2_control joint list, the DetachableJoint's
+       parent_link and the Clearpath/Franka includes; prefixing them would mean
+       touching all of those. Gazebo scopes links by model name already, and the
+       TF tree is separated by robot_state_publisher's frame_prefix - which is
+       exactly what the prefixed sensor frames above are matched to. See
+       tf_frame() in pick_and_place.py for the rule the mission code follows. -->
+  <xacro:arg name="robot_ns" default=""/>
+  <xacro:property name="robot_ns" value="$(arg robot_ns)"/>
+  <!-- '' or '/r1' for topic names; '' or 'r1/' for frame ids. -->
+  <xacro:property name="ns_topic" value="${'' if robot_ns == '' else '/' + robot_ns}"/>
+  <xacro:property name="ns_frame" value="${'' if robot_ns == '' else robot_ns + '/'}"/>
   <xacro:property name="PI" value="3.14159265359"/>
   <!-- Materials for the sensor housings we add ourselves (the A200 and FR3

Commit message: Step 4.1: Faster scenario. Main remaining issue is in placing

File: src/pickplace_arm_description/urdf/pickplace_arm.gazebo.xacro (robot description, xacro)
@@ -294,20 +294,69 @@
     <sensor name="lidar" type="gpu_lidar">
       <topic>${ns_topic}/scan</topic>
-      <update_rate>10</update_rate>
+      <!-- 15 Hz, up from 10. THIS SCAN IS NOW THE FLEET'S ANTI COLLISION
+           SENSE, not just a wall finder, and a closing speed matters to it.
+           Two robots approaching head on at the raised 0.90 m/s vx_max close
+           0.18 m between frames at 10 Hz and 0.12 m at 15 Hz. The local costmap
+           is raised to 15 Hz alongside it (nav2_params.yaml), so every costmap
+           update now has a scan it has not already seen, which is what makes
+           the avoidance FASTER rather than merely better informed.
+           IT IS ALSO THE CHEAPEST PLACE IN THIS SYSTEM TO SPEND. A gpu_lidar is
+           rendered on the GPU, which sits near idle on this machine while the
+           CPU is the thing that runs out, and the ROS side cost is a LaserScan
+           of a few hundred floats against the ~33 MB/s per robot the RGB-D
+           clouds already push through one bridge. -->
+      <update_rate>15</update_rate>
       <always_on>1</always_on>
       <visualize>true</visualize>
       <lidar>
         <scan>
-          <!-- 270 deg forward arc (-135..+135 deg); the excluded 90 deg
-               wedge points straight back at the arm, so the scan never hits
-               it. With the FR3 at x=0.0799 and this sensor at x=0.4449 the
-               arm subtends only ~+/-21 deg about the 180 deg bearing, well
-               inside the wedge. 270 samples keeps the same ~1 deg/sample
-               resolution as a 360-sample full circle. -->
+          <!-- 190 deg forward arc (-95..+95 deg), DOWN FROM 270, and the cut is
+               forced by the mount rather than chosen.
+               Hung under the plate the sensor scans at 0.3143 m, which is
+               chassis height, so for the first time the robot's own body is in
+               the scan plane. Two things are in it, and both were sliced out of
+               the meshes rather than guessed. From the laser centre at
+               base_link x=0.4100:
+                 front wheels   cross section at this height is x 0.185..0.327,
+                                y 0.220..0.335 (a cylinder cut off axis). Its
+                                forward outer corner bears 104.0 deg.
+                 chassis        tapers to x=0.3268, y +/-0.2104 here. Its front
+                                corner bears 111.6 deg.
+               So everything past 104 deg is the robot looking at itself. Those
+               hits are not harmlessly short either. Measured on one robot alone
+               on an empty ground plane with this mount and the old 270 deg arc:
+                   beams   1..46   bearing -134.5 .. -112.0 deg   0.184..0.362 m
+                   beams 494..539  bearing +112.5 .. +135.0 deg   0.172..0.357 m
+               (that run had the sensor 45 mm further forward, which is why its
+               boundary is 112 deg rather than 104 - the same model predicts
+               111.0 for it, so the model is good to about a beam). 92 of 540
+               beams reporting a solid obstacle a quarter of a metre away, above
+               range_min so nothing downstream filters them: a permanent phantom
+               wall in both costmaps and a block of beams AMCL can never match.
+               95 deg keeps 9 deg of margin to the wheel corner and is verified
+               empty: 0 of 380 beams return on a clear plane, and 34 of 380 - a
+               16.6 deg block at 2.21..2.33 m - when another robot stands 3 m
+               ahead.
+               WHAT IS GIVEN UP is the two rear quadrants; the blind sector goes
+               from 90 deg to 170. That is simply what a body height scanner on
+               the nose of a 0.99 m robot can see, and it buys the ability to
+               see other robots and the furniture AT ALL, which the 270 deg
+               version did not have.
+               270 samples over 190 deg = 0.70 deg, FINER than the 1.0 deg the
+               270 deg version had, on a third fewer beams. The things this
+               mount exists to detect are narrow - a table leg or a chair frame
+               subtends about 0.6 deg at 5 m and could fall between 1 deg beams
+               entirely - so the resolution matters and it improves here.
+               380 samples (0.5 deg) was tried and given back: the render is GPU
+               side and free, but every beam is raytraced into TWO costmaps per
+               robot, and at 15 Hz x 3 robots that is the difference between
+               4050 and 5700 rays a second of CPU. The real-time factor is what
+               the wall clock actually measures. AMCL subsamples to
+               max_beams=90 either way. -->
           <horizontal>
             <samples>270</samples>
             <resolution>1</resolution>
-            <min_angle>-2.35619449</min_angle>
-            <max_angle>2.35619449</max_angle>
+            <min_angle>-1.65806279</min_angle>
+            <max_angle>1.65806279</max_angle>
           </horizontal>
         </scan>

File: src/pickplace_arm_description/urdf/pickplace_arm.urdf.xacro (robot description, xacro)
@@ -241,14 +241,52 @@
   <!-- ==================================================================== -->
   <!-- ============ 2D LIDAR (SLAM / Nav2) ============
-       On the front of the top plate. The 270 deg forward arc configured in
-       pickplace_arm.gazebo.xacro excludes a 90 deg wedge pointing straight
-       BACK, which is exactly where the arm stands: the FR3 base is at
-       x=0.07987 and the LIDAR at x=0.40687, so the arm sits 0.327 m directly
-       behind the sensor and subtends only ~+/-15 deg there -comfortably
-       inside the excluded 135..225 deg wedge, so the scan never hits it.
-       HEIGHT CHANGED: this sits 0.447 m above the ground, against 0.11 m on
-       the old placeholder chassis. It now scans well above low obstacles,
-       so any ground-level box that SLAM/Nav2 used to see in the scan will no
-       longer appear. -->
+       HUNG UPSIDE DOWN, FULLY UNDER THE TOP PLATE.
+       WHAT WAS WRONG WITH STANDING IT ON THE PLATE. The scan plane sat 0.4467 m
+       above the floor. Every robot in this fleet is 0.3566 m tall at the top of
+       its chassis and 0.3836 m at the top of its plate, so a 2D scan at 0.4467
+       passed clean OVER the body of every other robot in the building. The only
+       part of a neighbour it could return was the FR3 tube standing on that
+       robot's plate. Measured, two robots 3 m apart facing each other:
+           standing on the plate, 0.4466 m    8 beams over  3.6 deg
+           hung under it,         0.3143 m   34 beams over 16.6 deg
+       Eight beams off a pole is not an obstacle a costmap can act on, which is
+       why three robots sharing a corridor were very nearly invisible to each
+       other. The same 0.4467 m plane also missed every table, trolley, bed
+       frame and chair seat in the hospital, and nav2_params.yaml gives the
+       costmaps this LIDAR and NOTHING ELSE as an obstacle source.
+       WHAT THE FLIP BUYS. rpy roll = pi turns the device over so it hangs from
+       the plate's underside instead of standing on its top. That drops the
+       laser centre by 0.1323 m in one move: 0.06296 to get from above the plate
+       to below it, twice, plus the plate's own 0.00639. The scan plane lands at
+       0.3143 m, inside the 0.1301..0.3566 m band the A200 chassis occupies, so
+       a neighbouring robot is now a solid body plus four wheels rather than a
+       stick.
+       WHY IT ALSO MOVES BACK 3.5 mm, AND WHY THAT IS THE INTERESTING NUMBER.
+       The device has to end up ENTIRELY under the plate, which is a window with
+       a wall at each end, both measured rather than assumed:
+         FRONT WALL  the plate's front edge is at x=0.4462 and the housing
+                     reaches 0.02903 ahead of the laser centre, so the laser
+                     centre cannot go past x=0.41717 without the scanner
+                     overhanging the lip into open air.
+         BACK WALL   the chassis is in the way. The housing hangs through
+                     base_link z 0.15914..0.245, and the A200's body TAPERS
+                     through that band: sliced off base_link.dae and
+                     top_chassis.dae it reaches x=0.3516 at z=0.159 and only
+                     0.2791 at z=0.220. The rear boss sits 0.04729 behind the
+                     laser centre, so the laser centre cannot come back past
+                     x=0.39889 without burying the boss in the chassis.
+       x=0.4100 sits in the middle of that 18 mm window: the housing spans
+       0.36271..0.43903, which is 7.2 mm inboard of the plate's lip and 11.1 mm
+       clear of the chassis. The old mount was at 0.40687 with the device
+       standing on top, so this is 3.5 mm further back and 0.1323 m lower.
+       THE ARM IS NO LONGER PART OF THIS. The old 90 deg rear wedge existed
+       because the FR3 stands 0.327 m behind the sensor at scan height. Below
+       the plate there is no arm in the plane at all, only the chassis and the
+       front wheels, and the arc in pickplace_arm.gazebo.xacro is cut to clear
+       those instead. See the note there for the measured bearings.
+       THE MAP MUST BE REGENERATED WITH THIS. aws_hospital_map.py builds the
+       Nav2 map by slicing the world at Z_LIDAR, so that constant and this joint
+       are one number in two places; a map sliced at a height the sensor does
+       not scan is a localisation failure, not a cosmetic one. -->
   <!-- Modelled as a SICK TiM5xx (TiM571): a real 270 deg, single-plane scanner
        whose datasheet geometry is what the sensor config above already
@@ -292,22 +330,37 @@
     <parent link="top_plate_front_mount"/>
     <child link="lidar_link"/>
-    <!-- Stand the real device ON the plate, fully INBOARD of its front edge.
-         Two corrections, both against the measured mesh envelope above:
-         z = +0.06296 (not SICK's 0.05595). lidar_link IS the laser centre and
-         the mesh's base plate is 0.06296 below it, so this puts the housing's
-         floor on the plate's upper surface (0.25135 in base_link) to within
-         0.1 mm. The old value buried the bottom 7 mm of the housing in the
-         plate. Scan plane: 0.4467 m above the floor, up from 0.4396.
-         x = -0.038. top_plate_front_mount sits at top_plate_link x=0.44487 but
-         the plate's front EDGE is at 0.4462 - only 1.3 mm further forward -
-         while the mesh reaches 0.02903 ahead of the laser centre. Mounted with
-         no x offset, 27.7 mm of the scanner hung off the front of the plate in
-         mid-air. Pulling it back 38 mm puts its front face at 0.4359, i.e.
-         10.3 mm inboard of the edge, with the whole footprint on the plate.
-         Neither change costs anything downstream: warehouse walls span the
-         full height either way, the carried box still rides 0.17 m clear above
-         the scan plane, and the arm stays deep inside the excluded rear wedge
-         (see above). -->
-    <origin xyz="-0.038 0 0.06296" rpy="0 0 0"/>
+    <!-- Hang the device UNDER the plate, inverted and wholly inboard. All three
+         numbers come from the measured mesh envelope above and the chassis
+         slices quoted in the block before this one.
+         rpy roll = pi. The device is turned over, so its base plate (0.06296
+         BELOW the laser centre in the mesh) now sits 0.06296 ABOVE it, bedded
+         against the plate's underside, and the optical head points down.
+         Rolling about X rather than Y is deliberate: it leaves +x forward, so
+         the scan arc stays symmetric about the bow and every bearing in the
+         sensor config keeps its meaning. Nothing downstream needs to know the
+         sensor is inverted. The LaserScan is published in lidar_link,
+         robot_state_publisher carries the roll in TF, and AMCL, the costmaps
+         and RViz all transform through it (nav2_amcl transforms angle_min and
+         the increment into the base frame precisely for this case).
+         z = -0.06935 = -(0.00639 + 0.06296). top_plate_front_mount sits on the
+         plate's UPPER surface; 0.00639 down reaches the underside at base_link
+         0.245, and the inverted device beds flat against it, putting the laser
+         centre 0.06296 lower still at base_link 0.18204 - 0.3143 m above the
+         floor.
+         x = -0.03487, i.e. base_link 0.4100. This is the "fully under the
+         plate" constraint and it is a two sided one: the housing must not
+         overhang the plate's lip at 0.4462 (laser centre <= 0.41717) and its
+         rear boss must not enter the tapering chassis, which reaches 0.3516 at
+         the housing's lowest point (laser centre >= 0.39889). 0.4100 is
+         centred in that window, leaving 7.2 mm to the lip and 11.1 mm to the
+         chassis. It is also inside the chassis collision box's own 0.4937, so
+         the robot's physical envelope is unchanged.
+         WHAT THIS COSTS. The carried payload has to clear a plane 0.1323 m
+         LOWER, which is slack rather than cost - carry_height() in
+         pick_and_place.py re-derives it from LIDAR_SCAN_Z. What it does cost is
+         the rear of the old 270 deg arc, which at this height is the robot's
+         own wheels and chassis; that trade is argued and measured in
+         pickplace_arm.gazebo.xacro, where the arc is set. -->
+    <origin xyz="-0.03487 0 -0.06935" rpy="${PI} 0 0"/>
   </joint>
   <!-- IMU: its yaw is fused with the wheel odometry (robot_localization EKF)
